File: Photogrammetry Plate.kicad_pro.kicad_pcb (KiCad board)
At the start: 2 copper layers, 280 x 280 mm, 32 parts

Commit message: New layout ready for order
Parts:
- removed the REF** at (320.0, 100.0)
- removed the REF** at (320.0, 180.0)
- removed the REF** at (360.0, 100.0)
- removed the REF** at (360.0, 180.0)
- removed the REF** at (360.0, 140.0)
- removed the REF** at (400.0, 260.0)
- removed the REF** at (280.0, 100.0)
- removed the REF** at (400.0, 220.0)
- removed the REF** at (200.0, 180.0)
- removed the REF** at (320.0, 220.0)
- removed the REF** at (320.0, 260.0)
- removed the REF** at (400.0, 180.0)
- removed the REF** at (280.0, 220.0)
- removed the REF** at (280.0, 140.0)
- removed the REF** at (240.0, 300.0)
- removed the REF** at (320.0, 140.0)
- removed the REF** at (240.0, 260.0)
- removed the REF** at (200.0, 260.0)
- removed the REF** at (360.0, 220.0)
- removed the REF** at (240.0, 220.0)
- removed the REF** at (400.0, 140.0)
- removed the REF** at (280.0, 180.0)
- removed the REF** at (360.0, 300.0)
- removed the REF** at (280.0, 300.0)
- removed the REF** at (240.0, 180.0)
- removed the REF** at (360.0, 260.0)
- removed the REF** at (320.0, 300.0)
- removed the REF** at (240.0, 140.0)
- removed the REF** at (200.0, 140.0)
- added REF**1: CCTAG_0015, CCTags:CCTAG_0015, F.Cu at (257.9, 98.4)
- added REF**10: CCTAG_0006, CCTags:CCTAG_0006, F.Cu at (377.8, 277.8)
- added REF**11: CCTAG_0005, CCTags:CCTAG_0005, F.Cu at (401.6, 242.1)
- added REF**12: CCTAG_0004, CCTags:CCTAG_0004, F.Cu at (410.0, 200.0)
- added REF**13: CCTAG_0003, CCTags:CCTAG_0003, F.Cu at (401.6, 157.9)
- added REF**14: CCTAG_0002, CCTags:CCTAG_0002, F.Cu at (377.8, 122.2)
- added REF**15: CCTAG_0001, CCTags:CCTAG_0001, F.Cu at (342.1, 98.4)
- added REF**16: CCTAG_0023, CCTags:CCTAG_0023, F.Cu at (250.5, 150.5)
- added REF**17: CCTAG_0022, CCTags:CCTAG_0022, F.Cu at (230.0, 200.0)
- added REF**18: CCTAG_0021, CCTags:CCTAG_0021, F.Cu at (250.5, 249.5)
- added REF**19: CCTAG_0020, CCTags:CCTAG_0020, F.Cu at (300.0, 270.0)
- added REF**2: CCTAG_0014, CCTags:CCTAG_0014, F.Cu at (222.2, 122.2)
- added REF**20: CCTAG_0019, CCTags:CCTAG_0019, F.Cu at (349.5, 249.5)
- added REF**21: CCTAG_0018, CCTags:CCTAG_0018, F.Cu at (370.0, 200.0)
- added REF**22: CCTAG_0017, CCTags:CCTAG_0017, F.Cu at (349.5, 150.5)
- added REF**23: CCTAG_0027, CCTags:CCTAG_0027, F.Cu at (270.0, 200.0)
- added REF**24: CCTAG_0026, CCTags:CCTAG_0026, F.Cu at (300.0, 230.0)
- added REF**25: CCTAG_0025, CCTags:CCTAG_0025, F.Cu at (330.0, 200.0)
- added REF**3: CCTAG_0013, CCTags:CCTAG_0013, F.Cu at (198.4, 157.9)
- added REF**4: CCTAG_0012, CCTags:CCTAG_0012, F.Cu at (190.0, 200.0)
- added REF**5: CCTAG_0011, CCTags:CCTAG_0011, F.Cu at (198.4, 242.1)
- added REF**6: CCTAG_0010, CCTags:CCTAG_0010, F.Cu at (222.2, 277.8)
- added REF**7: CCTAG_0009, CCTags:CCTAG_0009, F.Cu at (257.9, 301.6)
- added REF**8: CCTAG_0008, CCTags:CCTAG_0008, F.Cu at (300.0, 310.0)
- added REF**9: CCTAG_0007, CCTags:CCTAG_0007, F.Cu at (342.1, 301.6)
- moved REF** 134.5 mm to (300.0, 130.0)
- moved REF** 92.2 mm to (300.0, 170.0)
- moved REF** 60.8 mm to (300.0, 90.0)
Routing:
- net (no net): vias 0 -> 4
Other:
- board size 280 x 280 mm -> 250 x 250 mm
